Commit message: fix: four wheel drive, nit: comments

File: software/model/ros2_ws/src/rover/urdf/rover.urdf (robot description, URDF)
Before this commit: robot rover, 14 links, 13 joints
Links:
- removed link wheel_mid_left
- removed link wheel_mid_right
Joints:
- removed joint wheel_mid_left_joint
- removed joint wheel_mid_right_joint
