Commit message: partial

File: software/model/ros2_ws/src/rover/description/gazebo_control.xacro (robot description, xacro)
@@ -2,5 +2,5 @@
 <robot xmlns:xacro="http://www.ros.org/wiki/xacro">
 	<gazebo>
-    	<plugin filename="libgazebo_ros2_control.so" name="gazebo_ros2_control">
+        <plugin name="gz_ros2_control::GazeboSimROS2ControlPlugin" filename="libgz_ros2_control-system.so">
       		<parameters>$(find rover)/config/controller_position.yaml</parameters>
     	</plugin>

File: software/model/ros2_ws/src/rover/description/rover_core_lr.xacro (robot description, xacro)
@@ -157,5 +157,5 @@
       <origin xyz="0 0 0" rpy="0 0 0"/>
       <geometry>
-        <mesh filename="../meshes/base_link.STL"/>
+        <mesh filename="/home/aagrawal05/URC2024/software/model/ros2_ws/src/rover/meshes/base_link.STL"/>
       </geometry>
       <material name="arm_gray"/>
@@ -164,5 +164,5 @@
       <origin xyz="0 0 0" rpy="0 0 0"/>
       <geometry>
-        <mesh filename="../meshes/base_link.STL"/>
+        <mesh filename="/home/aagrawal05/URC2024/software/model/ros2_ws/src/rover/meshes/base_link.STL"/>
       </geometry>
     </collision>
@@ -183,5 +183,5 @@
       <origin xyz="0 0 0" rpy="0 0 0"/>
       <geometry>
-        <mesh filename="../meshes/link1.STL"/>
+        <mesh filename="/home/aagrawal05/URC2024/software/model/ros2_ws/src/rover/meshes/link1.STL"/>
       </geometry>
       <material name="arm_gray"/>
@@ -190,5 +190,5 @@
       <origin xyz="0 0 0" rpy="0 0 0"/>
       <geometry>
-        <mesh filename="../meshes/link1.STL"/>
+        <mesh filename="/home/aagrawal05/URC2024/software/model/ros2_ws/src/rover/meshes/link1.STL"/>
       </geometry>
     </collision>
@@ -210,5 +210,5 @@
       <origin xyz="0 0 0" rpy="0 0 0"/>
       <geometry>
-        <mesh filename="../meshes/link2.STL"/>
+        <mesh filename="/home/aagrawal05/URC2024/software/model/ros2_ws/src/rover/meshes/link2.STL"/>
       </geometry>
       <material name="arm_gray"/>
@@ -217,5 +217,5 @@
       <origin xyz="0 0 0" rpy="0 0 0"/>
       <geometry>
-        <mesh filename="../meshes/link2.STL"/>
+        <mesh filename="/home/aagrawal05/URC2024/software/model/ros2_ws/src/rover/meshes/link2.STL"/>
       </geometry>
     </collision>
@@ -237,5 +237,5 @@
       <origin xyz="0 0 0" rpy="0 0 0"/>
       <geometry>
-        <mesh filename="../meshes/link3.STL"/>
+        <mesh filename="/home/aagrawal05/URC2024/software/model/ros2_ws/src/rover/meshes/link3.STL"/>
       </geometry>
       <material name="arm_gray"/>
@@ -244,5 +244,5 @@
       <origin xyz="0 0 0" rpy="0 0 0"/>
       <geometry>
-        <mesh filename="../meshes/link3.STL"/>
+        <mesh filename="/home/aagrawal05/URC2024/software/model/ros2_ws/src/rover/meshes/link3.STL"/>
       </geometry>
     </collision>
@@ -264,5 +264,5 @@
       <origin xyz="0 0 0" rpy="0 0 0"/>
       <geometry>
-        <mesh filename="../meshes/wrist_link.STL"/>
+        <mesh filename="/home/aagrawal05/URC2024/software/model/ros2_ws/src/rover/meshes/wrist_link.STL"/>
       </geometry>
       <material name="white"/>
@@ -271,5 +271,5 @@
       <origin xyz="0 0 0" rpy="0 0 0"/>
       <geometry>
-        <mesh filename="../meshes/wrist_link.STL"/>
+        <mesh filename="/home/aagrawal05/URC2024/software/model/ros2_ws/src/rover/meshes/wrist_link.STL"/>
       </geometry>
     </collision>
@@ -291,5 +291,5 @@
       <origin xyz="0 0 0" rpy="0 0 0"/>
       <geometry>
-        <mesh filename="../meshes/manipulator.STL"/>
+        <mesh filename="/home/aagrawal05/URC2024/software/model/ros2_ws/src/rover/meshes/manipulator.STL"/>
       </geometry>
       <material name="white"/>
@@ -298,5 +298,5 @@
       <origin xyz="0 0 0" rpy="0 0 0"/>
       <geometry>
-        <mesh filename="../meshes/manipulator.STL"/>
+        <mesh filename="/home/aagrawal05/URC2024/software/model/ros2_ws/src/rover/meshes/manipulator.STL"/>
       </geometry>
     </collision>
@@ -318,5 +318,5 @@
       <origin xyz="0 0 0" rpy="0 0 0"/>
       <geometry>
-        <mesh filename="../meshes/claw.STL"/>
+        <mesh filename="/home/aagrawal05/URC2024/software/model/ros2_ws/src/rover/meshes/claw.STL"/>
       </geometry>
       <material name="white"/>
@@ -325,5 +325,5 @@
       <origin xyz="0 0 0" rpy="0 0 0"/>
       <geometry>
-        <mesh filename="../meshes/claw.STL"/>
+        <mesh filename="/home/aagrawal05/URC2024/software/model/ros2_ws/src/rover/meshes/claw.STL"/>
       </geometry>
     </collision>
@@ -339,5 +339,5 @@
   <ros2_control name="GazeboSystem" type="system">
     <hardware>
-      <plugin>gazebo_ros2_control/GazeboSystem</plugin>
+      <plugin>gz_ros2_control/GazeboSystem</plugin>
     </hardware>
     <!-- Arm Joint Control -->
@@ -428,5 +428,5 @@
     <plugin name="gz_ros2_control::GazeboSimROS2ControlPlugin" filename="libgz_ros2_control-system.so">
     <!-- <plugin name="gazebo_ros2_control" filename="libgazebo_ros2_control.so"> -->
-      <parameters>$(find rover)/config/controller_config.yaml</parameters>
+        <parameters>/home/aagrawal05/URC2024/software/model/ros2_ws/src/rover/config/controller_position.yaml</parameters>
     </plugin>
   </gazebo>
@@ -445,5 +445,5 @@
   </gazebo>
   <gazebo reference="wheel_rear_right">
-    <material>Gazebo/Black</material>
+    j<material>Gazebo/Black</material>
   </gazebo>
 </robot>

Commit message: having gpu error?

File: software/model/ros2_ws/src/rover/description/gazebo_control.xacro (robot description, xacro)
@@ -2,5 +2,5 @@
 <robot xmlns:xacro="http://www.ros.org/wiki/xacro">
 	<gazebo>
-    	<plugin filename="libgazebo_ros2_control.so" name="gazebo_ros2_control">
+<plugin filename="libgz_ros2_control-system.so" name="gz_ros2_control::GazeboSimROS2ControlPlugin"/>
       		<parameters>$(find rover)/config/controller_position.yaml</parameters>
     	</plugin>

File: software/model/ros2_ws/src/rover/description/rover_core_lr.xacro (robot description, xacro)
@@ -157,5 +157,5 @@
       <origin xyz="0 0 0" rpy="0 0 0"/>
       <geometry>
-        <mesh filename="/home/spalo/URC2024/software/model/ros2_ws/src/rover/meshes/base_link.STL"/>
+        <mesh filename="/home/brandon/URC2024/software/model/ros2_ws/src/rover/meshes/base_link.STL"/>
       </geometry>
       <material name="arm_gray"/>
@@ -164,5 +164,5 @@
       <origin xyz="0 0 0" rpy="0 0 0"/>
       <geometry>
-        <mesh filename="/home/spalo/URC2024/software/model/ros2_ws/src/rover/meshes/base_link.STL"/>
+        <mesh filename="/home/brandon/URC2024/software/model/ros2_ws/src/rover/meshes/base_link.STL"/>
       </geometry>
     </collision>
@@ -183,5 +183,5 @@
       <origin xyz="0 0 0" rpy="0 0 0"/>
       <geometry>
-        <mesh filename="/home/spalo/URC2024/software/model/ros2_ws/src/rover/meshes/link1.STL"/>
+        <mesh filename="/home/brandon/URC2024/software/model/ros2_ws/src/rover/meshes/link1.STL"/>
       </geometry>
       <material name="arm_gray"/>
@@ -190,5 +190,5 @@
       <origin xyz="0 0 0" rpy="0 0 0"/>
       <geometry>
-        <mesh filename="/home/spalo/URC2024/software/model/ros2_ws/src/rover/meshes/link1.STL"/>
+        <mesh filename="/home/brandon/URC2024/software/model/ros2_ws/src/rover/meshes/link1.STL"/>
       </geometry>
     </collision>
@@ -210,5 +210,5 @@
       <origin xyz="0 0 0" rpy="0 0 0"/>
       <geometry>
-        <mesh filename="/home/spalo/URC2024/software/model/ros2_ws/src/rover/meshes/link2.STL"/>
+        <mesh filename="/home/brandon/URC2024/software/model/ros2_ws/src/rover/meshes/link2.STL"/>
       </geometry>
       <material name="arm_gray"/>
@@ -217,5 +217,5 @@
       <origin xyz="0 0 0" rpy="0 0 0"/>
       <geometry>
-        <mesh filename="/home/spalo/URC2024/software/model/ros2_ws/src/rover/meshes/link2.STL"/>
+        <mesh filename="/home/brandon/URC2024/software/model/ros2_ws/src/rover/meshes/link2.STL"/>
       </geometry>
     </collision>
@@ -237,5 +237,5 @@
       <origin xyz="0 0 0" rpy="0 0 0"/>
       <geometry>
-        <mesh filename="/home/spalo/URC2024/software/model/ros2_ws/src/rover/meshes/link3.STL"/>
+        <mesh filename="/home/brandon/URC2024/software/model/ros2_ws/src/rover/meshes/link3.STL"/>
       </geometry>
       <material name="arm_gray"/>
@@ -244,5 +244,5 @@
       <origin xyz="0 0 0" rpy="0 0 0"/>
       <geometry>
-        <mesh filename="/home/spalo/URC2024/software/model/ros2_ws/src/rover/meshes/link3.STL"/>
+        <mesh filename="/home/brandon/URC2024/software/model/ros2_ws/src/rover/meshes/link3.STL"/>
       </geometry>
     </collision>
@@ -264,5 +264,5 @@
       <origin xyz="0 0 0" rpy="0 0 0"/>
       <geometry>
-        <mesh filename="/home/spalo/URC2024/software/model/ros2_ws/src/rover/meshes/wrist_link.STL"/>
+        <mesh filename="/home/brandon/URC2024/software/model/ros2_ws/src/rover/meshes/wrist_link.STL"/>
       </geometry>
       <material name="white"/>
@@ -271,5 +271,5 @@
       <origin xyz="0 0 0" rpy="0 0 0"/>
       <geometry>
-        <mesh filename="/home/spalo/URC2024/software/model/ros2_ws/src/rover/meshes/wrist_link.STL"/>
+        <mesh filename="/home/brandon/URC2024/software/model/ros2_ws/src/rover/meshes/wrist_link.STL"/>
       </geometry>
     </collision>
@@ -291,5 +291,5 @@
       <origin xyz="0 0 0" rpy="0 0 0"/>
       <geometry>
-        <mesh filename="/home/spalo/URC2024/software/model/ros2_ws/src/rover/meshes/manipulator.STL"/>
+        <mesh filename="/home/brandon/URC2024/software/model/ros2_ws/src/rover/meshes/manipulator.STL"/>
       </geometry>
       <material name="white"/>
@@ -298,5 +298,5 @@
       <origin xyz="0 0 0" rpy="0 0 0"/>
       <geometry>
-        <mesh filename="/home/spalo/URC2024/software/model/ros2_ws/src/rover/meshes/manipulator.STL"/>
+        <mesh filename="/home/brandon/URC2024/software/model/ros2_ws/src/rover/meshes/manipulator.STL"/>
       </geometry>
     </collision>
@@ -318,5 +318,5 @@
       <origin xyz="0 0 0" rpy="0 0 0"/>
       <geometry>
-        <mesh filename="/home/spalo/URC2024/software/model/ros2_ws/src/rover/meshes/claw.STL"/>
+        <mesh filename="/home/brandon/URC2024/software/model/ros2_ws/src/rover/meshes/claw.STL"/>
       </geometry>
       <material name="white"/>
@@ -325,5 +325,5 @@
       <origin xyz="0 0 0" rpy="0 0 0"/>
       <geometry>
-        <mesh filename="/home/spalo/URC2024/software/model/ros2_ws/src/rover/meshes/claw.STL"/>
+        <mesh filename="/home/brandon/URC2024/software/model/ros2_ws/src/rover/meshes/claw.STL"/>
       </geometry>
     </collision>
