Commit message: feat: controllers on all joints, bug: mesh files unlocated

File: software/model/ros2_ws/src/rover/description/rover_core_lr.xacro (robot description, xacro)
@@ -1,26 +1,33 @@
 <?xml version="1.0"?>
-<!--
-  URDF for Arm_Final_PLease with a support base and 6 actuated wheels.
-  Wheels are placed along the long sides (x-axis) at y = ±0.35 and are connected with continuous joints.
-  The wheel geometry is rotated so that it rolls about the y-axis.
--->
-<robot name="rover">
+<robot xmlns:xacro="http://www.ros.org/wiki/xacro">
+  <!-- Define materials -->
+  <material name="gray">
+    <color rgba="0.5 0.5 0.5 1"/>
+  </material>
+  <material name="black">
+    <color rgba="0 0 0 1"/>
+  </material>
+  <material name="arm_gray">
+    <color rgba="0.792156862745098 0.819607843137255 0.933333333333333 1"/>
+  </material>
+  <material name="white">
+    <color rgba="1 1 1 1"/>
+  </material>
+  <material name="blue">
+    <color rgba="0.0 0.0 0.8 1"/>
+  </material>
   <!-- Define the support base as a new link -->
-  <link name="base_support">
-    <visual>
-      <origin xyz="0 0 0" rpy="0 0 0"/>
-      <geometry>
-        <!-- Visual dimensions of the support (can be adjusted as needed) -->
-        <box size="0.85 0.7 0.3"/>
-      </geometry>
-      <material name="gray">
-        <color rgba="0.5 0.5 0.5 1"/>
-      </material>
-    </visual>
-    <collision>
-      <origin xyz="0 0 0" rpy="0 0 0"/>
-      <geometry>
-        <!-- Collision box: using 1.3m x 0.7m x 0.1m dimensions -->
-        <box size="1.3 0.7 0.1"/>
+  <link name="chassis">
+    <visual>
+      <origin xyz="0 0 0" rpy="0 0 0"/>
+      <geometry>
+        <box size="0.704 0.46 0.216"/>
+      </geometry>
+      <material name="blue"/>
+    </visual>
+    <collision>
+      <origin xyz="0 0 0" rpy="0 0 0"/>
+      <geometry>
+        <box size="0.704 0.46 0.216"/>
       </geometry>
     </collision>
@@ -31,6 +38,7 @@
     </inertial>
   </link>
-  <!-- Define six wheel links (actuated wheels) -->
-  <!-- Each wheel is modeled as a cylinder with its visual and collision geometry rotated so that its axis aligns with the wheel rotation -->
+  <!-- Define four wheel links (actuated wheels) -->
+  <!-- Now front_left is actually rear_left, front_right is rear_right -->
+  <!-- And rear_left is front_left, rear_right is front_right -->
   <link name="wheel_front_left">
     <visual>
@@ -39,7 +47,5 @@
         <cylinder radius="0.1" length="0.05"/>
       </geometry>
-      <material name="black">
-        <color rgba="0 0 0 1"/>
-      </material>
+      <material name="black"/>
     </visual>
     <collision>
@@ -61,7 +67,5 @@
         <cylinder radius="0.1" length="0.05"/>
       </geometry>
-      <material name="black">
-        <color rgba="0 0 0 1"/>
-      </material>
+      <material name="black"/>
     </visual>
     <collision>
@@ -77,13 +81,11 @@
     </inertial>
   </link>
-  <link name="wheel_mid_left">
-    <visual>
-      <origin xyz="0 0 0" rpy="1.5708 0 0"/>
-      <geometry>
-        <cylinder radius="0.1" length="0.05"/>
-      </geometry>
-      <material name="black">
-        <color rgba="0 0 0 1"/>
-      </material>
+  <link name="wheel_rear_left">
+    <visual>
+      <origin xyz="0 0 0" rpy="1.5708 0 0"/>
+      <geometry>
+        <cylinder radius="0.1" length="0.05"/>
+      </geometry>
+      <material name="black"/>
     </visual>
     <collision>
@@ -99,13 +101,11 @@
     </inertial>
   </link>
-  <link name="wheel_mid_right">
-    <visual>
-      <origin xyz="0 0 0" rpy="1.5708 0 0"/>
-      <geometry>
-        <cylinder radius="0.1" length="0.05"/>
-      </geometry>
-      <material name="black">
-        <color rgba="0 0 0 1"/>
-      </material>
+  <link name="wheel_rear_right">
+    <visual>
+      <origin xyz="0 0 0" rpy="1.5708 0 0"/>
+      <geometry>
+        <cylinder radius="0.1" length="0.05"/>
+      </geometry>
+      <material name="black"/>
     </visual>
     <collision>
@@ -121,95 +121,29 @@
     </inertial>
   </link>
-  <link name="wheel_rear_left">
-    <visual>
-      <origin xyz="0 0 0" rpy="1.5708 0 0"/>
-      <geometry>
-        <cylinder radius="0.1" length="0.05"/>
-      </geometry>
-      <material name="black">
-        <color rgba="0 0 0 1"/>
-      </material>
-    </visual>
-    <collision>
-      <origin xyz="0 0 0" rpy="1.5708 0 0"/>
-      <geometry>
-        <cylinder radius="0.1" length="0.05"/>
-      </geometry>
-    </collision>
-    <inertial>
-      <origin xyz="0 0 0" rpy="0 0 0"/>
-      <mass value="0.5"/>
-      <inertia ixx="0.01" ixy="0" ixz="0" iyy="0.01" iyz="0" izz="0.01"/>
-    </inertial>
-  </link>
-  <link name="wheel_rear_right">
-    <visual>
-      <origin xyz="0 0 0" rpy="1.5708 0 0"/>
-      <geometry>
-        <cylinder radius="0.1" length="0.05"/>
-      </geometry>
-      <material name="black">
-        <color rgba="0 0 0 1"/>
-      </material>
-    </visual>
-    <collision>
-      <origin xyz="0 0 0" rpy="1.5708 0 0"/>
-      <geometry>
-        <cylinder radius="0.1" length="0.05"/>
-      </geometry>
-    </collision>
-    <inertial>
-      <origin xyz="0 0 0" rpy="0 0 0"/>
-      <mass value="0.5"/>
-      <inertia ixx="0.01" ixy="0" ixz="0" iyy="0.01" iyz="0" izz="0.01"/>
-    </inertial>
-  </link>
   <!-- Joints for attaching each wheel to the support base -->
-  <!-- Wheels are attached along the long sides at y = ±0.35.
-       The x positions (0.65, 0, -0.65) distribute them evenly along the 1.3m length.
-       The joint axis is set to 0 1 0 so that the wheel rotates about the y‑axis. -->
+  <!-- Rotated wheel positions: front becomes rear and rear becomes front -->
   <joint name="wheel_front_left_joint" type="continuous">
-    <parent link="base_support"/>
+    <parent link="chassis"/>
     <child link="wheel_front_left"/>
-    <origin xyz="0.55 0.40 -0.05" rpy="0 0 0"/>
+    <origin xyz="0.25 0.30 -0.05" rpy="0 0 0"/>
     <axis xyz="0 1 0"/>
   </joint>
   <joint name="wheel_front_right_joint" type="continuous">
-    <parent link="base_support"/>
+    <parent link="chassis"/>
     <child link="wheel_front_right"/>
-    <origin xyz="0.55 -0.40 -0.05" rpy="0 0 0"/>
+    <origin xyz="0.25 -0.30 -0.05" rpy="0 0 0"/>
     <axis xyz="0 1 0"/>
   </joint>
-  <joint name="wheel_mid_left_joint" type="continuous">
-    <parent link="base_support"/>
-    <child link="wheel_mid_left"/>
-    <origin xyz="0 0.40 -0.05" rpy="0 0 0"/>
+  <joint name="wheel_rear_left_joint" type="continuous">
+    <parent link="chassis"/>
+    <child link="wheel_rear_left"/>
+    <origin xyz="-0.25 0.30 -0.05" rpy="0 0 0"/>
     <axis xyz="0 1 0"/>
   </joint>
-  <joint name="wheel_mid_right_joint" type="continuous">
-    <parent link="base_support"/>
-    <child link="wheel_mid_right"/>
-    <origin xyz="0 -0.40 -0.05" rpy="0 0 0"/>
+  <joint name="wheel_rear_right_joint" type="continuous">
+    <parent link="chassis"/>
+    <child link="wheel_rear_right"/>
+    <origin xyz="-0.25 -0.30 -0.05" rpy="0 0 0"/>
     <axis xyz="0 1 0"/>
-  </joint>
-  <joint name="wheel_rear_left_joint" type="continuous">
-    <parent link="base_support"/>
-    <child link="wheel_rear_left"/>
-    <origin xyz="-0.55 0.40 -0.05" rpy="0 0 0"/>
-    <axis xyz="0 1 0"/>
-  </joint>
-  <joint name="wheel_rear_right_joint" type="continuous">
-    <parent link="base_support"/>
-    <child link="wheel_rear_right"/>
-    <origin xyz="-0.55 -0.40 -0.05" rpy="0 0 0"/>
-    <axis xyz="0 1 0"/>
-  </joint>
-  <!-- Attach the arm's base (base_link) to the support with a fixed joint.
-       The origin offset (0.0635, -0.0635, 0.05) compensates for the base_link inertial offset,
-       centering the arm on the support base. -->
-  <joint name="base_mount" type="fixed">
-    <parent link="base_support"/>
-    <child link="base_link"/>
-    <origin xyz="0.0635 -0.0635 0.05" rpy="0 0 0"/>
   </joint>
   <!-- Arm's URDF as previously defined -->
@@ -225,7 +159,5 @@
         <mesh filename="../meshes/base_link.STL"/>
       </geometry>
-      <material name="">
-        <color rgba="0.792156862745098 0.819607843137255 0.933333333333333 1"/>
-      </material>
+      <material name="arm_gray"/>
     </visual>
     <collision>
@@ -236,4 +168,10 @@
     </collision>
   </link>
+  <!-- Attach the arm's base (base_link) to the support with a fixed joint -->
+  <joint name="base_mount" type="fixed">
+    <parent link="chassis"/>
+    <child link="base_link"/>
+    <origin xyz="0.0635 -0.0635 0.15" rpy="0 0 0"/>
+  </joint>
   <link name="link1">
     <inertial>
@@ -247,7 +185,5 @@
         <mesh filename="../meshes/link1.STL"/>
       </geometry>
-      <material name="">
-        <color rgba="0.792156862745098 0.819607843137255 0.933333333333333 1"/>
-      </material>
+      <material name="arm_gray"/>
     </visual>
     <collision>
@@ -276,7 +212,5 @@
         <mesh filename="../meshes/link2.STL"/>
       </geometry>
-      <material name="">
-        <color rgba="0.792156862745098 0.819607843137255 0.933333333333333 1"/>
-      </material>
+      <material name="arm_gray"/>
     </visual>
     <collision>
@@ -305,7 +239,5 @@
         <mesh filename="../meshes/link3.STL"/>
       </geometry>
-      <material name="">
-        <color rgba="0.792156862745098 0.819607843137255 0.933333333333333 1"/>
-      </material>
+      <material name="arm_gray"/>
     </visual>
     <collision>
@@ -334,7 +266,5 @@
         <mesh filename="../meshes/wrist_link.STL"/>
       </geometry>
-      <material name="">
-        <color rgba="0.898039215686275 0.917647058823529 0.929411764705882 1"/>
-      </material>
+      <material name="white"/>
     </visual>
     <collision>
@@ -363,7 +293,5 @@
         <mesh filename="../meshes/manipulator.STL"/>
       </geometry>
-      <material name="">
-        <color rgba="1 1 1 1"/>
-      </material>
+      <material name="white"/>
     </visual>
     <collision>
@@ -392,12 +320,10 @@
         <mesh filename="../meshes/claw.STL"/>
       </geometry>
-      <material name="">
-        <color rgba="1 1 1 1"/>
-      </material>
-    </visual>
-    <collision>
-      <origin xyz="0 0 0" rpy="0 0 0"/>
-      <geometry>
-	      <mesh filename="../meshes/claw.STL"/>
+      <material name="white"/>
+    </visual>
+    <collision>
+      <origin xyz="0 0 0" rpy="0 0 0"/>
+      <geometry>
+        <mesh filename="../meshes/claw.STL"/>
       </geometry>
     </collision>
@@ -410,3 +336,113 @@
     <limit lower="-0.1425" upper="0" effort="100" velocity="1"/>
   </joint>
+  <!-- ROS2 Control Integration -->
+  <ros2_control name="GazeboSystem" type="system">
+    <hardware>
+      <plugin>gazebo_ros2_control/GazeboSystem</plugin>
+    </hardware>
+    <!-- Arm Joint Control -->
+    <joint name="platform">
+      <command_interface name="position">
+        <param name="min">-3.1416</param>
+        <param name="max">3.1416</param>
+      </command_interface>
+      <state_interface name="position"/>
+      <state_interface name="velocity"/>
+    </joint>
+    <joint name="linkage1">
+      <command_interface name="position">
+        <param name="min">-3.1416</param>
+        <param name="max">3.1416</param>
+      </command_interface>
+      <state_interface name="position"/>
+      <state_interface name="velocity"/>
+    </joint>
+    <joint name="linkage3">
+      <command_interface name="position">
+        <param name="min">-3.1416</param>
+        <param name="max">3.1416</param>
+      </command_interface>
+      <state_interface name="position"/>
+      <state_interface name="velocity"/>
+    </joint>
+    <joint name="wrist">
+      <command_interface name="position">
+        <param name="min">-3.1416</param>
+        <param name="max">3.1416</param>
+      </command_interface>
+      <state_interface name="position"/>
+      <state_interface name="velocity"/>
+    </joint>
+    <joint name="manipulator_wrist">
+      <command_interface name="position">
+        <param name="min">-3.1416</param>
+        <param name="max">3.1416</param>
+      </command_interface>
+      <state_interface name="position"/>
+      <state_interface name="velocity"/>
+    </joint>
+    <joint name="top_claw">
+      <command_interface name="position">
+        <param name="min">-0.1425</param>
+        <param name="max">0</param>
+      </command_interface>
+      <state_interface name="position"/>
+      <state_interface name="velocity"/>
+    </joint>
+    <!-- Wheel Control -->
+    <joint name="wheel_front_left_joint">
+      <command_interface name="velocity">
+        <param name="min">-10</param>
+        <param name="max">10</param>
+      </command_interface>
+      <state_interface name="position"/>
+      <state_interface name="velocity"/>
+    </joint>
+    <joint name="wheel_front_right_joint">
+      <command_interface name="velocity">
+        <param name="min">-10</param>
+        <param name="max">10</param>
+      </command_interface>
+      <state_interface name="position"/>
+      <state_interface name="velocity"/>
+    </joint>
+    <joint name="wheel_rear_left_joint">
+      <command_interface name="velocity">
+        <param name="min">-10</param>
+        <param name="max">10</param>
+      </command_interface>
+      <state_interface name="position"/>
+      <state_interface name="velocity"/>
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
Commit message: The file changes for jazzy->humble, untested as my humble gazebo does not work yet

File: software/model/ros2_ws/src/rover/description/rover_core_lr.xacro (robot description, xacro)
@@ -157,5 +157,5 @@
       <origin xyz="0 0 0" rpy="0 0 0"/>
       <geometry>
-        <mesh filename="/home/spalo/URC2024/software/model/ros2_ws/src/rover/meshes/base_link.STL"/>
+        <mesh filename="/home/brandon/URC2024/software/model/ros2_ws/src/rover/meshes/base_link.STL"/>
       </geometry>
       <material name="arm_gray"/>
@@ -164,5 +164,5 @@
       <origin xyz="0 0 0" rpy="0 0 0"/>
       <geometry>
-        <mesh filename="/home/spalo/URC2024/software/model/ros2_ws/src/rover/meshes/base_link.STL"/>
+        <mesh filename="/home/brandon/URC2024/software/model/ros2_ws/src/rover/meshes/base_link.STL"/>
       </geometry>
     </collision>
@@ -183,5 +183,5 @@
       <origin xyz="0 0 0" rpy="0 0 0"/>
       <geometry>
-        <mesh filename="/home/spalo/URC2024/software/model/ros2_ws/src/rover/meshes/link1.STL"/>
+        <mesh filename="/home/brandon/URC2024/software/model/ros2_ws/src/rover/meshes/link1.STL"/>
       </geometry>
       <material name="arm_gray"/>
@@ -190,5 +190,5 @@
       <origin xyz="0 0 0" rpy="0 0 0"/>
       <geometry>
-        <mesh filename="/home/spalo/URC2024/software/model/ros2_ws/src/rover/meshes/link1.STL"/>
+        <mesh filename="/home/brandon/URC2024/software/model/ros2_ws/src/rover/meshes/link1.STL"/>
       </geometry>
     </collision>
@@ -210,5 +210,5 @@
       <origin xyz="0 0 0" rpy="0 0 0"/>
       <geometry>
-        <mesh filename="/home/spalo/URC2024/software/model/ros2_ws/src/rover/meshes/link2.STL"/>
+        <mesh filename="/home/brandon/URC2024/software/model/ros2_ws/src/rover/meshes/link2.STL"/>
       </geometry>
       <material name="arm_gray"/>
@@ -217,5 +217,5 @@
       <origin xyz="0 0 0" rpy="0 0 0"/>
       <geometry>
-        <mesh filename="/home/spalo/URC2024/software/model/ros2_ws/src/rover/meshes/link2.STL"/>
+        <mesh filename="/home/brandon/URC2024/software/model/ros2_ws/src/rover/meshes/link2.STL"/>
       </geometry>
     </collision>
@@ -237,5 +237,5 @@
       <origin xyz="0 0 0" rpy="0 0 0"/>
       <geometry>
-        <mesh filename="/home/spalo/URC2024/software/model/ros2_ws/src/rover/meshes/link3.STL"/>
+        <mesh filename="/home/brandon/URC2024/software/model/ros2_ws/src/rover/meshes/link3.STL"/>
       </geometry>
       <material name="arm_gray"/>
@@ -244,5 +244,5 @@
       <origin xyz="0 0 0" rpy="0 0 0"/>
       <geometry>
-        <mesh filename="/home/spalo/URC2024/software/model/ros2_ws/src/rover/meshes/link3.STL"/>
+        <mesh filename="/home/brandon/URC2024/software/model/ros2_ws/src/rover/meshes/link3.STL"/>
       </geometry>
     </collision>
@@ -264,5 +264,5 @@
       <origin xyz="0 0 0" rpy="0 0 0"/>
       <geometry>
-        <mesh filename="/home/spalo/URC2024/software/model/ros2_ws/src/rover/meshes/wrist_link.STL"/>
+        <mesh filename="/home/brandon/URC2024/software/model/ros2_ws/src/rover/meshes/wrist_link.STL"/>
       </geometry>
       <material name="white"/>
@@ -271,5 +271,5 @@
       <origin xyz="0 0 0" rpy="0 0 0"/>
       <geometry>
-        <mesh filename="/home/spalo/URC2024/software/model/ros2_ws/src/rover/meshes/wrist_link.STL"/>
+        <mesh filename="/home/brandon/URC2024/software/model/ros2_ws/src/rover/meshes/wrist_link.STL"/>
       </geometry>
     </collision>
@@ -291,5 +291,5 @@
       <origin xyz="0 0 0" rpy="0 0 0"/>
       <geometry>
-        <mesh filename="/home/spalo/URC2024/software/model/ros2_ws/src/rover/meshes/manipulator.STL"/>
+        <mesh filename="/home/brandon/URC2024/software/model/ros2_ws/src/rover/meshes/manipulator.STL"/>
       </geometry>
       <material name="white"/>
@@ -298,5 +298,5 @@
       <origin xyz="0 0 0" rpy="0 0 0"/>
       <geometry>
-        <mesh filename="/home/spalo/URC2024/software/model/ros2_ws/src/rover/meshes/manipulator.STL"/>
+        <mesh filename="/home/brandon/URC2024/software/model/ros2_ws/src/rover/meshes/manipulator.STL"/>
       </geometry>
     </collision>
@@ -318,5 +318,5 @@
       <origin xyz="0 0 0" rpy="0 0 0"/>
       <geometry>
-        <mesh filename="/home/spalo/URC2024/software/model/ros2_ws/src/rover/meshes/claw.STL"/>
+        <mesh filename="/home/brandon/URC2024/software/model/ros2_ws/src/rover/meshes/claw.STL"/>
       </geometry>
       <material name="white"/>
@@ -325,5 +325,5 @@
       <origin xyz="0 0 0" rpy="0 0 0"/>
       <geometry>
-        <mesh filename="/home/spalo/URC2024/software/model/ros2_ws/src/rover/meshes/claw.STL"/>
+        <mesh filename="/home/brandon/URC2024/software/model/ros2_ws/src/rover/meshes/claw.STL"/>
       </geometry>
     </collision>
@@ -339,5 +339,5 @@
   <ros2_control name="GazeboSystem" type="system">
     <hardware>
-      <plugin>gz_ros2_control/GazeboSimSystem</plugin>
+      <plugin>gazebo_ros2_control/GazeboSystem</plugin>
     </hardware>
     <!-- Arm Joint Control -->
@@ -426,5 +426,5 @@
   <!-- Gazebo plugin for ROS 2 control -->
   <gazebo>
-     <plugin name="gz_ros2_control::GazeboSimROS2ControlPlugin" filename="libgz_ros2_control-system.so">
+    <plugin name="gazebo_ros2_control" filename="libgazebo_ros2_control.so">
       <parameters>$(find rover)/config/controller_position.yaml</parameters>
     </plugin>

Commit message: feat: movit config and basic implemenation path planning

File: software/model/ros2_ws/src/rover/description/rover_core_lr.xacro (robot description, xacro)
@@ -157,5 +157,5 @@
       <origin xyz="0 0 0" rpy="0 0 0"/>
       <geometry>
-        <mesh filename="/home/brandon/URC2024/software/model/ros2_ws/src/rover/meshes/base_link.STL"/>
+        <mesh filename="package://rover/meshes/base_link.STL"/>
       </geometry>
       <material name="arm_gray"/>
@@ -164,5 +164,5 @@
       <origin xyz="0 0 0" rpy="0 0 0"/>
       <geometry>
-        <mesh filename="/home/brandon/URC2024/software/model/ros2_ws/src/rover/meshes/base_link.STL"/>
+        <mesh filename="package://rover/meshes/base_link.STL"/>
       </geometry>
     </collision>
@@ -183,5 +183,5 @@
       <origin xyz="0 0 0" rpy="0 0 0"/>
       <geometry>
-        <mesh filename="/home/brandon/URC2024/software/model/ros2_ws/src/rover/meshes/link1.STL"/>
+        <mesh filename="package://rover/meshes/link1.STL"/>
       </geometry>
       <material name="arm_gray"/>
@@ -190,5 +190,5 @@
       <origin xyz="0 0 0" rpy="0 0 0"/>
       <geometry>
-        <mesh filename="/home/brandon/URC2024/software/model/ros2_ws/src/rover/meshes/link1.STL"/>
+        <mesh filename="package://rover/meshes/link1.STL"/>
       </geometry>
     </collision>
@@ -210,5 +210,5 @@
       <origin xyz="0 0 0" rpy="0 0 0"/>
       <geometry>
-        <mesh filename="/home/brandon/URC2024/software/model/ros2_ws/src/rover/meshes/link2.STL"/>
+        <mesh filename="package://rover/meshes/link2.STL"/>
       </geometry>
       <material name="arm_gray"/>
@@ -217,5 +217,5 @@
       <origin xyz="0 0 0" rpy="0 0 0"/>
       <geometry>
-        <mesh filename="/home/brandon/URC2024/software/model/ros2_ws/src/rover/meshes/link2.STL"/>
+        <mesh filename="package://rover/meshes/link2.STL"/>
       </geometry>
     </collision>
@@ -237,5 +237,5 @@
       <origin xyz="0 0 0" rpy="0 0 0"/>
       <geometry>
-        <mesh filename="/home/brandon/URC2024/software/model/ros2_ws/src/rover/meshes/link3.STL"/>
+        <mesh filename="package://rover/meshes/link3.STL"/>
       </geometry>
       <material name="arm_gray"/>
@@ -244,5 +244,5 @@
       <origin xyz="0 0 0" rpy="0 0 0"/>
       <geometry>
-        <mesh filename="/home/brandon/URC2024/software/model/ros2_ws/src/rover/meshes/link3.STL"/>
+        <mesh filename="package://rover/meshes/link3.STL"/>
       </geometry>
     </collision>
@@ -264,5 +264,5 @@
       <origin xyz="0 0 0" rpy="0 0 0"/>
       <geometry>
-        <mesh filename="/home/brandon/URC2024/software/model/ros2_ws/src/rover/meshes/wrist_link.STL"/>
+        <mesh filename="package://rover/meshes/wrist_link.STL"/>
       </geometry>
       <material name="white"/>
@@ -271,5 +271,5 @@
       <origin xyz="0 0 0" rpy="0 0 0"/>
       <geometry>
-        <mesh filename="/home/brandon/URC2024/software/model/ros2_ws/src/rover/meshes/wrist_link.STL"/>
+        <mesh filename="package://rover/meshes/wrist_link.STL"/>
       </geometry>
     </collision>
@@ -291,5 +291,5 @@
       <origin xyz="0 0 0" rpy="0 0 0"/>
       <geometry>
-        <mesh filename="/home/brandon/URC2024/software/model/ros2_ws/src/rover/meshes/manipulator.STL"/>
+        <mesh filename="package://rover/meshes/manipulator.STL"/>
       </geometry>
       <material name="white"/>
@@ -298,5 +298,5 @@
       <origin xyz="0 0 0" rpy="0 0 0"/>
       <geometry>
-        <mesh filename="/home/brandon/URC2024/software/model/ros2_ws/src/rover/meshes/manipulator.STL"/>
+        <mesh filename="package://rover/meshes/manipulator.STL"/>
       </geometry>
     </collision>
@@ -318,5 +318,5 @@
       <origin xyz="0 0 0" rpy="0 0 0"/>
       <geometry>
-        <mesh filename="/home/brandon/URC2024/software/model/ros2_ws/src/rover/meshes/claw.STL"/>
+        <mesh filename="package://rover/meshes/claw.STL"/>
       </geometry>
       <material name="white"/>
@@ -325,5 +325,5 @@
       <origin xyz="0 0 0" rpy="0 0 0"/>
       <geometry>
-        <mesh filename="/home/brandon/URC2024/software/model/ros2_ws/src/rover/meshes/claw.STL"/>
+        <mesh filename="package://rover/meshes/claw.STL"/>
       </geometry>
     </collision>
