Commit message: feat: created sequence of stretch movement

File: software/model/ros2_ws/src/rover/description/rover_core_lr.xacro (robot description, xacro)
@@ -157,5 +157,5 @@
       <origin xyz="0 0 0" rpy="0 0 0"/>
       <geometry>
-        <mesh filename="/home/brandon/URC2024/software/model/ros2_ws/src/rover/meshes/base_link.STL"/>
+        <mesh filename="/home/spalo/URC2024/software/model/ros2_ws/src/rover/meshes/base_link.STL"/>
       </geometry>
       <material name="arm_gray"/>
@@ -164,5 +164,5 @@
       <origin xyz="0 0 0" rpy="0 0 0"/>
       <geometry>
-        <mesh filename="/home/brandon/URC2024/software/model/ros2_ws/src/rover/meshes/base_link.STL"/>
+        <mesh filename="/home/spalo/URC2024/software/model/ros2_ws/src/rover/meshes/base_link.STL"/>
       </geometry>
     </collision>
@@ -183,5 +183,5 @@
       <origin xyz="0 0 0" rpy="0 0 0"/>
       <geometry>
-        <mesh filename="/home/brandon/URC2024/software/model/ros2_ws/src/rover/meshes/link1.STL"/>
+        <mesh filename="/home/spalo/URC2024/software/model/ros2_ws/src/rover/meshes/link1.STL"/>
       </geometry>
       <material name="arm_gray"/>
@@ -190,5 +190,5 @@
       <origin xyz="0 0 0" rpy="0 0 0"/>
       <geometry>
-        <mesh filename="/home/brandon/URC2024/software/model/ros2_ws/src/rover/meshes/link1.STL"/>
+        <mesh filename="/home/spalo/URC2024/software/model/ros2_ws/src/rover/meshes/link1.STL"/>
       </geometry>
     </collision>
@@ -210,5 +210,5 @@
       <origin xyz="0 0 0" rpy="0 0 0"/>
       <geometry>
-        <mesh filename="/home/brandon/URC2024/software/model/ros2_ws/src/rover/meshes/link2.STL"/>
+        <mesh filename="/home/spalo/URC2024/software/model/ros2_ws/src/rover/meshes/link2.STL"/>
       </geometry>
       <material name="arm_gray"/>
@@ -217,5 +217,5 @@
       <origin xyz="0 0 0" rpy="0 0 0"/>
       <geometry>
-        <mesh filename="/home/brandon/URC2024/software/model/ros2_ws/src/rover/meshes/link2.STL"/>
+        <mesh filename="/home/spalo/URC2024/software/model/ros2_ws/src/rover/meshes/link2.STL"/>
       </geometry>
     </collision>
@@ -237,5 +237,5 @@
       <origin xyz="0 0 0" rpy="0 0 0"/>
       <geometry>
-        <mesh filename="/home/brandon/URC2024/software/model/ros2_ws/src/rover/meshes/link3.STL"/>
+        <mesh filename="/home/spalo/URC2024/software/model/ros2_ws/src/rover/meshes/link3.STL"/>
       </geometry>
       <material name="arm_gray"/>
@@ -244,5 +244,5 @@
       <origin xyz="0 0 0" rpy="0 0 0"/>
       <geometry>
-        <mesh filename="/home/brandon/URC2024/software/model/ros2_ws/src/rover/meshes/link3.STL"/>
+        <mesh filename="/home/spalo/URC2024/software/model/ros2_ws/src/rover/meshes/link3.STL"/>
       </geometry>
     </collision>
@@ -264,5 +264,5 @@
       <origin xyz="0 0 0" rpy="0 0 0"/>
       <geometry>
-        <mesh filename="/home/brandon/URC2024/software/model/ros2_ws/src/rover/meshes/wrist_link.STL"/>
+        <mesh filename="/home/spalo/URC2024/software/model/ros2_ws/src/rover/meshes/wrist_link.STL"/>
       </geometry>
       <material name="white"/>
@@ -271,5 +271,5 @@
       <origin xyz="0 0 0" rpy="0 0 0"/>
       <geometry>
-        <mesh filename="/home/brandon/URC2024/software/model/ros2_ws/src/rover/meshes/wrist_link.STL"/>
+        <mesh filename="/home/spalo/URC2024/software/model/ros2_ws/src/rover/meshes/wrist_link.STL"/>
       </geometry>
     </collision>
@@ -291,5 +291,5 @@
       <origin xyz="0 0 0" rpy="0 0 0"/>
       <geometry>
-        <mesh filename="/home/brandon/URC2024/software/model/ros2_ws/src/rover/meshes/manipulator.STL"/>
+        <mesh filename="/home/spalo/URC2024/software/model/ros2_ws/src/rover/meshes/manipulator.STL"/>
       </geometry>
       <material name="white"/>
@@ -298,5 +298,5 @@
       <origin xyz="0 0 0" rpy="0 0 0"/>
       <geometry>
-        <mesh filename="/home/brandon/URC2024/software/model/ros2_ws/src/rover/meshes/manipulator.STL"/>
+        <mesh filename="/home/spalo/URC2024/software/model/ros2_ws/src/rover/meshes/manipulator.STL"/>
       </geometry>
     </collision>
@@ -318,5 +318,5 @@
       <origin xyz="0 0 0" rpy="0 0 0"/>
       <geometry>
-        <mesh filename="/home/brandon/URC2024/software/model/ros2_ws/src/rover/meshes/claw.STL"/>
+        <mesh filename="/home/spalo/URC2024/software/model/ros2_ws/src/rover/meshes/claw.STL"/>
       </geometry>
       <material name="white"/>
@@ -325,5 +325,5 @@
       <origin xyz="0 0 0" rpy="0 0 0"/>
       <geometry>
-        <mesh filename="/home/brandon/URC2024/software/model/ros2_ws/src/rover/meshes/claw.STL"/>
+        <mesh filename="/home/spalo/URC2024/software/model/ros2_ws/src/rover/meshes/claw.STL"/>
       </geometry>
     </collision>

Commit message: Fixed package scope

File: software/model/ros2_ws/src/rover/description/rover_core_lr.xacro (robot description, xacro)
@@ -157,5 +157,5 @@
       <origin xyz="0 0 0" rpy="0 0 0"/>
       <geometry>
-        <mesh filename="package://rover/meshes/base_link.STL"/>
+        <mesh filename="package://src/rover/meshes/base_link.STL"/>
       </geometry>
       <material name="arm_gray"/>
@@ -164,5 +164,5 @@
       <origin xyz="0 0 0" rpy="0 0 0"/>
       <geometry>
-        <mesh filename="package://rover/meshes/base_link.STL"/>
+        <mesh filename="package://src/rover/meshes/base_link.STL"/>
       </geometry>
     </collision>
@@ -183,5 +183,5 @@
       <origin xyz="0 0 0" rpy="0 0 0"/>
       <geometry>
-        <mesh filename="package://rover/meshes/link1.STL"/>
+        <mesh filename="package://src/rover/meshes/link1.STL"/>
       </geometry>
       <material name="arm_gray"/>
@@ -190,5 +190,5 @@
       <origin xyz="0 0 0" rpy="0 0 0"/>
       <geometry>
-        <mesh filename="package://rover/meshes/link1.STL"/>
+        <mesh filename="package://src/rover/meshes/link1.STL"/>
       </geometry>
     </collision>
@@ -210,5 +210,5 @@
       <origin xyz="0 0 0" rpy="0 0 0"/>
       <geometry>
-        <mesh filename="package://rover/meshes/link2.STL"/>
+        <mesh filename="package://src/rover/meshes/link2.STL"/>
       </geometry>
       <material name="arm_gray"/>
@@ -217,5 +217,5 @@
       <origin xyz="0 0 0" rpy="0 0 0"/>
       <geometry>
-        <mesh filename="package://rover/meshes/link2.STL"/>
+        <mesh filename="package://src/rover/meshes/link2.STL"/>
       </geometry>
     </collision>
@@ -237,5 +237,5 @@
       <origin xyz="0 0 0" rpy="0 0 0"/>
       <geometry>
-        <mesh filename="package://rover/meshes/link3.STL"/>
+        <mesh filename="package://src/rover/meshes/link3.STL"/>
       </geometry>
       <material name="arm_gray"/>
@@ -244,5 +244,5 @@
       <origin xyz="0 0 0" rpy="0 0 0"/>
       <geometry>
-        <mesh filename="package://rover/meshes/link3.STL"/>
+        <mesh filename="package://src/rover/meshes/link3.STL"/>
       </geometry>
     </collision>
@@ -264,5 +264,5 @@
       <origin xyz="0 0 0" rpy="0 0 0"/>
       <geometry>
-        <mesh filename="package://rover/meshes/wrist_link.STL"/>
+        <mesh filename="package://src/rover/meshes/wrist_link.STL"/>
       </geometry>
       <material name="white"/>
@@ -271,5 +271,5 @@
       <origin xyz="0 0 0" rpy="0 0 0"/>
       <geometry>
-        <mesh filename="package://rover/meshes/wrist_link.STL"/>
+        <mesh filename="package://src/rover/meshes/wrist_link.STL"/>
       </geometry>
     </collision>
@@ -291,5 +291,5 @@
       <origin xyz="0 0 0" rpy="0 0 0"/>
       <geometry>
-        <mesh filename="package://rover/meshes/manipulator.STL"/>
+        <mesh filename="package://src/rover/meshes/manipulator.STL"/>
       </geometry>
       <material name="white"/>
@@ -298,5 +298,5 @@
       <origin xyz="0 0 0" rpy="0 0 0"/>
       <geometry>
-        <mesh filename="package://rover/meshes/manipulator.STL"/>
+        <mesh filename="package://src/rover/meshes/manipulator.STL"/>
       </geometry>
     </collision>
@@ -318,5 +318,5 @@
       <origin xyz="0 0 0" rpy="0 0 0"/>
       <geometry>
-        <mesh filename="package://rover/meshes/claw.STL"/>
+        <mesh filename="package://src/rover/meshes/claw.STL"/>
       </geometry>
       <material name="white"/>
@@ -325,5 +325,5 @@
       <origin xyz="0 0 0" rpy="0 0 0"/>
       <geometry>
-        <mesh filename="package://rover/meshes/claw.STL"/>
+        <mesh filename="package://src/rover/meshes/claw.STL"/>
       </geometry>
     </collision>
